File: Hardware/RedBot Whisker Bumper.sch (EAGLE design)
At the start: 9 parts

Commit message: Production Readied
Parts:
- added FID1, FID2: FIDUCIALUFIDUCIAL, SparkFun-Aesthetics:FIDUCIALUFIDUCIAL
Changed lines of the file:
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@@
 <part name="LOGO3" library="SparkFun-Aesthetics" deviceset="OSHW-LOGO" device="S"/>
 <part name="LOGO4" library="SparkFun-Aesthetics" deviceset="LOGO-SFE" device="SK"/>
+<part name="FID1" library="SparkFun-Aesthetics" deviceset="FIDUCIAL" device="UFIDUCIAL"/>
+<part name="FID2" library="SparkFun-Aesthetics" deviceset="FIDUCIAL" device="UFIDUCIAL"/>
 </parts>
 <sheets>
@@
 <instance part="LOGO3" gate="G$1" x="236.22" y="45.72"/>
 <instance part="LOGO4" gate="G$1" x="241.3" y="17.78"/>
+<instance part="FID1" gate="G$1" x="243.84" y="33.02"/>
+<instance part="FID2" gate="G$1" x="243.84" y="27.94"/>
 </instances>
 <busses>

Commit message: QC Revision
Changes:
1.) New 3-pin SMD header footprints w/ bosses
2.) Moved R1 position and routing for better reflow
Parts:
- JP1: device SparkFun-Connectors:M03SMD_RA_MALE -> SparkFun-Connectors:M03SMD_RA_MALE_POST
Other:
- note added: "Revision: Kade Jensen"
- note added: "v11"
- note removed: "v10"
Changed lines of the file:
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@@
 <?xml version="1.0" encoding="utf-8"?>
 <!DOCTYPE eagle SYSTEM "eagle.dtd">
-<eagle version="6.4">
+<eagle version="6.5.0">
 <drawing>
 <settings>
@@
 <layer number="18" name="Vias" color="2" fill="1" visible="no" active="no"/>
 <layer number="19" name="Unrouted" color="6" fill="1" visible="no" active="no"/>
-<layer number="20" name="Dimension" color="15" fill="1" visible="no" active="no"/>
-<layer number="21" name="tPlace" color="7" fill="1" visible="no" active="no"/>
-<layer number="22" name="bPlace" color="7" fill="1" visible="no" active="no"/>
+<layer number="20" name="Dimension" color="6" fill="1" visible="no" active="no"/>
+<layer number="21" name="tPlace" color="16" fill="1" visible="no" active="no"/>
+<layer number="22" name="bPlace" color="14" fill="1" visible="no" active="no"/>
 <layer number="23" name="tOrigins" color="15" fill="1" visible="no" active="no"/>
 <layer number="24" name="bOrigins" color="15" fill="1" visible="no" active="no"/>
@@
 <layer number="49" name="Reference" color="7" fill="1" visible="no" active="no"/>
 <layer number="50" name="dxf" color="7" fill="1" visible="no" active="no"/>
-<layer number="51" name="tDocu" color="7" fill="1" visible="no" active="no"/>
+<layer number="51" name="tDocu" color="6" fill="1" visible="no" active="no"/>
 <layer number="52" name="bDocu" color="7" fill="1" visible="no" active="no"/>
 <layer number="53" name="tGND_GNDA" color="7" fill="9" visible="no" active="no"/>
@@
 <layer number="106" name="bPlate" color="7" fill="1" visible="no" active="yes"/>
 <layer number="107" name="Crop" color="7" fill="1" visible="no" active="yes"/>
+<layer number="108" name="tplace-old" color="10" fill="1" visible="yes" active="yes"/>
+<layer number="109" name="ref-old" color="11" fill="1" visible="yes" active="yes"/>
 <layer number="116" name="Patch_BOT" color="9" fill="4" visible="no" active="yes"/>
 <layer number="121" name="_tsilk" color="7" fill="1" visible="no" active="yes"/>
@@
 <part name="LOGO1" library="SparkFun-Aesthetics" deviceset="OSHW-LOGO" device="S"/>
 <part name="LOGO2" library="SparkFun-Aesthetics" deviceset="LOGO-SFE" device="SK"/>
-<part name="JP1" library="SparkFun-Connectors" deviceset="M03" device="SMD_RA_MALE"/>
+<part name="JP1" library="SparkFun-Connectors" deviceset="M03" device="SMD_RA_MALE_POST"/>
 <part name="R1" library="SparkFun-Resistors" deviceset="10KOHM1/10W1%(0603)" device="0603" value="10K"/>
 <part name="S1" library="SparkFun-Electromechanical" deviceset="STANDOFF_ELECTRICAL" device=""/>
@@
 <sheet>
 <plain>
-<text x="172.72" y="7.62" size="3.81" layer="94">M. Hord</text>
-<text x="237.49" y="6.35" size="3.81" layer="94">v10</text>
+<text x="170.434" y="11.43" size="2.54" layer="94">M. Hord</text>
+<text x="237.49" y="6.35" size="3.81" layer="94">v11</text>
+<text x="148.59" y="7.62" size="2.54" layer="94">Revision: Kade Jensen</text>
 </plain>
 <instances>
